Commit message: added in link to world joint

File: URDF/my_robot.urdf.xacro (robot description, xacro)
@@ -43,8 +43,8 @@
     </link>
     <!-- Define the joints -->
-    <joint name="joint1" type="fixed">
-        <parent link="base_link" />
-        <child link="wheel1" />
-        <origin xyz="0.25 0.25 0" rpy="0 0 0" />
+    <joint name="world_to_base" type="fixed">
+        <parent link="world" />
+        <child link="base_link" />
+        <origin xyz="0 0 0" rpy="0 0 0" />
     </joint>
     <joint name="joint2" type="fixed">

Commit message: applied materials

File: URDF/my_robot.urdf.xacro (robot description, xacro)
@@ -11,4 +11,5 @@
                 <box size="0.5 0.5 0.1" />
             </geometry>
+            <material name="red" />
         </visual>
     </link>
@@ -19,4 +20,5 @@
                 <cylinder length="0.1" radius="0.05" />
             </geometry>
+            <material name="black" />
         </visual>
     </link>
@@ -26,4 +28,5 @@
                 <cylinder length="0.1" radius="0.05" />
             </geometry>
+            <material name="black" />
         </visual>
     </link>
@@ -33,4 +36,5 @@
                 <cylinder length="0.1" radius="0.05" />
             </geometry>
+            <material name="black" />
         </visual>
     </link>
@@ -40,4 +44,5 @@
                 <cylinder length="0.1" radius="0.05" />
             </geometry>
+            <material name="black" />
         </visual>
     </link>

Commit message: added in the joint to the first wheel (strangely missing)

File: URDF/my_robot.urdf.xacro (robot description, xacro)
@@ -53,4 +53,9 @@
         <origin xyz="0 0 0" rpy="0 0 0" />
     </joint>
+    <joint name="joint1" type="fixed">
+        <parent link="base_link" />
+        <child link="wheel1" />
+        <origin xyz="0.25 0.25 0" rpy="0 0 0" />
+    </joint>
     <joint name="joint2" type="fixed">
         <parent link="base_link" />
